File: DMX512toWS2811.kicad_pcb (KiCad board)
At the start: 2 copper layers, 140 x 110 mm, 122 parts, among them CN1 TB112-2-2-E-1, CN2 18742, CN3 B6B-PH-K-S_LF__SN_, CN4 TB111-2-3-U-1-1, CN5 TB112-2-2-E-1, CN6 TB112-2-2-E-1, IC1 MAX485ESA+, IC2 MAX485ESA+, IC3 TLP2361_TPL,E, IC4 TCK106AF,LF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

Commit message: * ローカル保存分と同期
Parts:
- removed NT2, NTe: NetTie_2, NetTie:NetTie-2_SMD_Pad2.0mm
- removed the TP1 at (160.8, 71.5)
- removed the TP2 at (159.2, 69.5)
- added C20: 0.1u, Capacitor_SMD:C_0603_1608Metric_Pad1.08x0.95mm_HandSolder, F.Cu at (176.8, 61.8)
- added C21: 1000p, Capacitor_SMD:C_0603_1608Metric_Pad1.08x0.95mm_HandSolder, F.Cu at (176.0, 68.2)
- added CN7: TB112-2-2-E-1, SamacSys_Parts:TB11222E1, F.Cu at (189.5, 75.9)
- added IC8: NJU77551F-TE1, SamacSys_Parts:SOT95P280X130-5N, F.Cu at (176.2, 64.5)
- added R41: 2k, Resistor_SMD:R_0603_1608Metric_Pad0.98x0.95mm_HandSolder, F.Cu at (178.8, 67.5)
- added R42: 2k, Resistor_SMD:R_0603_1608Metric_Pad0.98x0.95mm_HandSolder, F.Cu at (178.8, 69.2)
- added R44: 0, Resistor_SMD:R_0603_1608Metric_Pad0.98x0.95mm_HandSolder, F.Cu at (173.2, 64.5)
- added R45: 10k, Resistor_SMD:R_0603_1608Metric_Pad0.98x0.95mm_HandSolder, F.Cu at (171.5, 61.0)
- added R46: 10k, Resistor_SMD:R_0603_1608Metric_Pad0.98x0.95mm_HandSolder, F.Cu at (171.5, 66.0)
- CN4: value TB111-2-3-U-1-1 -> TB112-2-2-E-1; footprint SamacSys_Parts:TB11123U11 -> SamacSys_Parts:TB11222E1
- moved CN3 42.7 mm to (151.5, 71.2)
- moved R35 32.3 mm to (132.8, 61.5), turned to 180 degrees
- moved C18 11.3 mm to (158.5, 57.5), turned to 90 degrees
- moved R30 8.75 mm to (158.5, 62.0), turned to -90 degrees
- moved R34 8.56 mm to (172.2, 54.2), turned to 0 degrees
- moved D4 8.33 mm to (180.2, 55.5), turned to -90 degrees
- moved TP3 6.19 mm to (159.0, 67.0)
- moved R29 5.95 mm to (166.5, 66.2), turned to 90 degrees
- moved CN4 5.18 mm to (189.5, 65.8)
- moved IC6 5.06 mm to (163.0, 59.5), turned to 90 degrees
- moved F3 4.90 mm to (181.5, 62.8), turned to -90 degrees
- moved R33 4.16 mm to (161.8, 113.8), turned to -90 degrees
- moved TP2 3.26 mm to (159.5, 69.8)
- moved R17 2.88 mm to (111.8, 81.0)
- moved C13 2.88 mm to (117.0, 78.2)
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- renumbered TP3 to TP1, TP4 to TP2, TP5 to TP3
Connections:
- CN4 pad 1: GND2 -> /WS_SIG_OUT
- CN4 pad 2: /SIG_OUT -> /5V_OUT
- CN6 pad 1: GND1 -> GND
- F3 pad 2: /SIG_OUT -> /WS_SIG_OUT
- IC5 pad 14: UART_RX -> 485_nRE
- IC5 pad 16: 485_nRE -> UART_RX
- IC5 pad 21: 5VOUT_EN -> OSIG_P
- IC5 pad 22: Net-(IC5-RB1) -> OSIG_N
- IC5 pad 23: Net-(IC5-RB2) -> 5VOUT_EN
Routing:
- net VDC: track 149.4 -> 22.8 mm
- net /5V_OUT: track 70.8 -> 0.00 mm
- net GND2: track 64.5 -> 0.00 mm
- net GND1: track 62.1 -> 0.00 mm
- net +5V: track 328.7 -> 272.5 mm
- net Net-(Q1-G): track 57.4 -> 7.73 mm, vias 4 -> 0
- net 5VOUT_EN: track 3.47 -> 51.0 mm, vias 0 -> 2
- net GND: track 200.4 -> 234.4 mm, vias 208 -> 48
- net VPP: track 31.6 -> 0.00 mm
- net ICSPDAT: track 42.4 -> 11.9 mm, vias 2 -> 0
- net 485_nRE: track 79.8 -> 50.7 mm
- net RESET: track 49.8 -> 21.3 mm
- net PSMODE_SW: track 87.2 -> 115.6 mm
- net ICSPCLK: track 41.1 -> 14.4 mm, vias 2 -> 0
- net OSIG_N: track 0.00 -> 22.9 mm, vias 0 -> 2
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- added copper zone on F.Cu, net +5V
- added copper zone on F.Cu, net /5V_OUT
- added copper zone on F.Cu, net Net-(D8-A)
- added copper zone on F.Cu, net VDC
- added copper zone on F.Cu, net VPP
Other:
- outline, holes or cut-outs redrawn
- board text added: "DO_O"
- board text added: "DO_W"
- board text removed: "DOUT"
