File: DMX512toWS2811.kicad_sch (KiCad schematic)
At the start: 122 parts, among them CN1 TB112-2-2-E-1, CN2 18742, CN3 B6B-PH-K-S_LF__SN_, CN4 TB111-2-3-U-1-1, CN5 TB112-2-2-E-1, CN6 TB112-2-2-E-1, IC1 MAX485ESA+, IC2 MAX485ESA+, IC3 TLP2361_TPL,E, IC4 TCK106AF,LF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

Commit message: * ローカル保存分と同期
Parts:
- removed CN4: TB111-2-3-U-1-1, TB11123U11, symbol SamacSys_Parts:TB111-2-3-U-1-1
- removed NT1, NT2: NetTie_2, NetTie:NetTie-2_SMD_Pad2.0mm, symbol Device:NetTie_2
- removed TP1, TP2: TestPoint, TestPoint:TestPoint_THTPad_D1.5mm_Drill0.7mm, symbol Connector:TestPoint
- added C20: 0.1u, Capacitor_SMD:C_0603_1608Metric_Pad1.08x0.95mm_HandSolder, symbol Device:C
- added C21: 1000p, Capacitor_SMD:C_0603_1608Metric_Pad1.08x0.95mm_HandSolder, symbol Device:C
- added CN4, CN7: TB112-2-2-E-1, TB11222E1, symbol SamacSys_Parts:TB112-2-2-E-1
- added IC8: NJU77551F-TE1, SOT95P280X130-5N, symbol SamacSys_Parts:NJU77551F-TE1
- added R41, R42: 2k, Resistor_SMD:R_0603_1608Metric_Pad0.98x0.95mm_HandSolder, symbol Device:R
- added R44: 0, Resistor_SMD:R_0603_1608Metric_Pad0.98x0.95mm_HandSolder, symbol Device:R
- added R45, R46: 10k, Resistor_SMD:R_0603_1608Metric_Pad0.98x0.95mm_HandSolder, symbol Device:R
- renumbered TP3 to TP1, TP4 to TP2, TP5 to TP3
Connections:
- net GND1 is gone; now on net GND: CN6.1
- net +5V: now also C20.2, IC8.5 (V+)
- net 485_nRE: now also IC5.14 (RC3); no longer IC5.16 (RC5)
- net 5VOUT_EN: now also IC5.23 (RB2); no longer IC5.21 (RB0)
- net 5V_OUT: now also CN4.2
- net GND: now also C20.1, CN7.1, IC8.2 (V-), R44.1
- net UART_RX: now also IC5.16 (RC5); no longer IC5.14 (RC3)
- net OSIG_N: now reaches IC5.22 (RB1)
- net OSIG_N: now also R45.1
- net SIG_OUT renamed WS_SIG_OUT
- net WS_SIG_OUT: now also CN4.1
- new net: IC8.1 (+INPUT), R44.2, R45.2, R46.2
- new net: C21.2, IC8.3 (-INPUT), R42.1
- new net: C21.1, IC8.4 (OUTPUT), R41.1
- new net OSIG_P: IC5.21 (RB0), R46.1
- new net OSRAM_SIG_OUT: CN7.2, R41.2, R42.2
Other:
- moved on the sheet: C10, C18, C8, CA1, CA3, CA4, CN1, CN2, CN3, D4, D6, F1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
